Commit message: tmp update 1229

File: src/universal-robot/realsense2_description/urdf/_d415.gazebo.xacro (robot description, xacro)
@@ -8,5 +8,5 @@
   <xacro:macro name="gazebo_d415" params="camera_name reference_link topics_ns depth_optical_frame color_optical_frame infrared1_optical_frame infrared2_optical_frame publish_pointcloud:=true" >
     <!-- Load parameters to model's main link-->
-    <xacro:property name="deg_to_rad" value="0.01745329251994329577" />
+    <!-- <xacro:property name="deg_to_rad" value="0.01745329251994329577" />
     <gazebo reference="${reference_link}">
       <self_collide>0</self_collide>
@@ -14,13 +14,13 @@
       <kinematic>0</kinematic>
       <gravity>1</gravity>
-      <!--<mu>1</mu>-->
+      <mu>1</mu>
       <mu2>1</mu2>
       <fdir1>0 0 0</fdir1>
-      <!--<slip1>0</slip1>
-      <slip2>0</slip2>-->
+      <slip1>0</slip1>
+      <slip2>0</slip2>
       <kp>1e+13</kp>
       <kd>1</kd>
-      <!--<max_vel>0.01</max_vel>
-      <min_depth>0</min_depth>-->
+      <max_vel>0.01</max_vel>
+      <min_depth>0</min_depth>
       <sensor name="${camera_name}color" type="camera">
         <camera name="${camera_name}">
@@ -136,5 +136,5 @@
         <pointCloudCutoffMax>9.0</pointCloudCutoffMax>
       </plugin>
-    </gazebo>
+    </gazebo> -->
   </xacro:macro>
 </robot>

File: src/universal-robot/realsense2_description/urdf/_d415.urdf.xacro (robot description, xacro)
@@ -117,4 +117,11 @@
     </joint>
     <link name="${name}_color_optical_frame"/>
+    <joint name="${name}_color_moveit_joint" type="fixed">
+      <!-- <origin xyz="0 0 0" rpy="${3*M_PI/2} 0 ${-M_PI/2}" /> -->
+      <origin xyz="0 0 0" rpy="${M_PI} ${-M_PI/2} 0" />
+      <parent link="${name}_color_frame" />
+      <child link="${name}_color_moveit_frame" />
+    </joint>
+    <link name="${name}_color_moveit_frame"/>
     <!-- Realsense Gazebo Plugin -->
     <xacro:gazebo_d415 camera_name="${name}" reference_link="${name}_link" topics_ns="${topics_ns}" depth_optical_frame="${name}_depth_optical_frame" color_optical_frame="${name}_color_optical_frame" infrared1_optical_frame="${name}_left_ir_optical_frame" infrared2_optical_frame="${name}_right_ir_optical_frame" publish_pointcloud="${publish_pointcloud}"/>
