Commit message: modified tcp urdf

File: src/universal-robot/ur_description/urdf/inc/ur5e_real_macro.xacro (robot description, xacro)
@@ -71,5 +71,5 @@
       <parent link="${prefix}wrist_3_link" />
       <child link="gripper_tcp" />
-      <origin xyz="0 0 0.2" rpy="0 0 0" />
+      <origin xyz="0 0 0.17" rpy="0 0 0" />
     </joint>
     <!-- camera -->

File: src/universal-robot/ur_description/urdf/inc/ur5e_sim_macro.xacro (robot description, xacro)
@@ -71,5 +71,5 @@
       <parent link="${prefix}wrist_3_link" />
       <child link="gripper_tcp" />
-      <origin xyz="0 0 0.2" rpy="0 0 0" />
+      <origin xyz="0 0 0.17" rpy="0 0 0" />
     </joint>
     <!-- camera -->

Commit message: change tcp depth

File: src/universal-robot/ur_description/urdf/inc/ur5e_real_macro.xacro (robot description, xacro)
@@ -71,5 +71,5 @@
       <parent link="${prefix}wrist_3_link" />
       <child link="gripper_tcp" />
-      <origin xyz="0 0 0.17" rpy="0 0 0" />
+      <origin xyz="0 0 0.155" rpy="0 0 0" />
     </joint>
     <!-- camera -->

File: src/universal-robot/ur_description/urdf/inc/ur5e_sim_macro.xacro (robot description, xacro)
@@ -71,5 +71,5 @@
       <parent link="${prefix}wrist_3_link" />
       <child link="gripper_tcp" />
-      <origin xyz="0 0 0.17" rpy="0 0 0" />
+      <origin xyz="0 0 0.155" rpy="0 0 0" />
     </joint>
     <!-- camera -->

Commit message: update 1128

File: src/universal-robot/ur_description/urdf/inc/ur5e_real_macro.xacro (robot description, xacro)
@@ -71,5 +71,5 @@
       <parent link="${prefix}wrist_3_link" />
       <child link="gripper_tcp" />
-      <origin xyz="0 0 0.155" rpy="0 0 0" />
+      <origin xyz="0 0 0.18" rpy="0 0 0" />
     </joint>
     <!-- camera -->
