Commit message: changed gripper_tcp link rotation

File: src/universal-robot/ur_description/urdf/inc/ur5e_sim_macro.xacro (robot description, xacro)
@@ -71,5 +71,5 @@
       <parent link="${prefix}wrist_3_link" />
       <child link="gripper_tcp" />
-      <origin xyz="0 0 0.155" rpy="0 0 0" />
+      <origin xyz="0 0 0.155" rpy="0 0 -1.57" />
     </joint>
     <!-- camera -->
